File: PCB/PCB_Turbina_V1/PCB_V2/PCB_V1.kicad_pcb (KiCad board)
At the start: 2 copper layers, 194 x 80 mm, 13 parts, among them J1 BATT_11.1V, J2 Conn_01x07, J3 ENODER_LEFT, J4 ENODER_RIGH, J5 BATT_7.4V, J6 JST-7.7V, J7 TURBINE_POWER, J8 TURBINE_PWM, SW1 Switch, U1 WeMos_S2_mini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

Commit message: Correccion V1
Parts:
- moved U3 2.12 mm to (222.7, 99.3)
- moved J4 2.12 mm to (215.2, 86.0)
Routing:
- net PWM_RIGH: track 174.1 -> 171.0 mm
- net OUTA_RIGH: track 128.3 -> 126.1 mm
- net GND: track 545.8 -> 547.9 mm
- net IN2_RIGH: track 160.0 -> 157.9 mm
- net STBY_RIGH: track 130.4 -> 131.1 mm
- net IN1_RIGH: track 144.9 -> 145.6 mm
- net (no net): vias 8 -> 12
Other:
- outline, holes or cut-outs redrawn
